File: INKTIME_PCB.brd (EAGLE design)
At the start: 46 x 35 mm, 103 parts, among them IC1 BQ25180YBGR, IC2 RT6160AWSC, IC3 BMA423, IC4 DRV2605YZFR, J1 503480-2400, J2 TC2030-IDC, J4 KH-TYPE-C-16P, Q1 SI1308EDL-T1-GE3, U1 NRF52840_QF, U3 MAX17048G+T10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

Commit message: fix issue 1
Parts:
- ANT1: device InkTime_v5:2450AT18B100E_ANTC3216X140N -> InkTime_v5v3:2450AT18B100E_ANTC3216X140N
- C1-EP-DR, C2-EP-DR, C25, C33, C43, EPD_C1, EPD_C10, EPD_C11, EPD_C12, EPD_C2, EPD_C5, EPD_C6, EPD_C7, EPD_C8, EPD_C9: device InkTime_v5:NORDIC_NRF_3_RESC0603_N -> InkTime_v5v3:NORDIC_NRF_3_RESC0603_N
- C10, C11, C12, C13, C17, C18, C19, C22, C3, C4, C5, C7, C8, C9, XC1, XC2: device InkTime_v5:NORDIC_NRF_3_RESC0201_L -> InkTime_v5v3:NORDIC_NRF_3_RESC0201_L
- C14, C16, C20, C21, C39, C6: device InkTime_v5:PERFECT_0402_0402 -> InkTime_v5v3:PERFECT_0402_0402
- C15: device InkTime_v5:NORDIC_NRF_3_RESC0402_L -> InkTime_v5v3:NORDIC_NRF_3_RESC0402_L
- C23: device InkTime_v5:GRM011R60J152KE01L_2_CAPC0201X13N -> InkTime_v5v3:GRM011R60J152KE01L_2_CAPC0201X13N
- C24: device InkTime_v5:NORDIC_NRF_3_RESC0402_N -> InkTime_v5v3:NORDIC_NRF_3_RESC0402_N
- C27, C29, C30, C31, C32, C34, C37, C38, C42: device InkTime_v5:GRM011R60J152KE01L_1_0201 -> InkTime_v5v3:GRM011R60J152KE01L_1_0201
- D2, D4, D5: device InkTime_v5:ESP32_C6_LIBRARY_5_SOD3716X135N -> InkTime_v5v3:ESP32_C6_LIBRARY_5_SOD3716X135N
- D3: device InkTime_v5:ESP32_C6_LIBRARY_3_SOT95P280X145-6N -> InkTime_v5v3:ESP32_C6_LIBRARY_3_SOT95P280X145-6N
- DMG2305UX-7: device InkTime_v5:ESP32_C6_LIBRARY_4_ESP32_C6_LIBRARY_4_ESP32_C6_LIBRARY_4_ESP32_C6_LIBRARY_4_ESP32_WROVER_SPARKFUN-DISCRETESE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 -> InkTime_v5v3:ESP32_C6_LIBRARY_4_ESP32_C6_LIBRARY_4_ESP32_C6_LIBRARY_4_ESP32_C6_LIBRARY_4_ESP32_WROVER_SPARKFUN-DISCRETE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
- IC1: device InkTime_v5:BQ25180YBGR_BGA8C40P2X4_100X155X50 -> InkTime_v5v3:BQ25180YBGR_BGA8C40P2X4_100X155X50
- IC2: device InkTime_v5:RT6160AWSC_BGA15C40P3X5_140X230X60 -> InkTime_v5v3:RT6160AWSC_BGA15C40P3X5_140X230X60
- IC3: device InkTime_v5:BMA423_BMA423 -> InkTime_v5v3:BMA423_BMA423
- IC4: device InkTime_v5:DRV2605YZFR_BGA9C50P3X3_144X144X62 -> InkTime_v5v3:DRV2605YZFR_BGA9C50P3X3_144X144X62
- J1: device InkTime_v5:503480-2400_5034802400 -> InkTime_v5v3:503480-2400_5034802400
- J2: device InkTime_v5:TC2030-IDC_TC2030IDC -> InkTime_v5v3:TC2030-IDC_TC2030IDC
- J4: device InkTime_v5v2:KH-TYPE-C-16P_KINGHELM_KH-TYPE-C-16P -> InkTime_v5v3:KH-TYPE-C-16P_KINGHELM_KH-TYPE-C-16P
- L1, L2, L3: device InkTime_v5:NORDIC_NRF_2_RESC0201_L -> InkTime_v5v3:NORDIC_NRF_2_RESC0201_L
- L5: device InkTime_v5:ESP32_C6_LIBRARY_2_IND_4828-WE-TPC_WRE -> InkTime_v5v3:ESP32_C6_LIBRARY_2_IND_4828-WE-TPC_WRE
- L7: device InkTime_v5:MLP2016SR47MT0S1_INDC2016X100N -> InkTime_v5v3:MLP2016SR47MT0S1_INDC2016X100N
- Q1: device InkTime_v5:ESP32_C6_LIBRARY_6_SOT65P210X110-3N -> InkTime_v5v3:ESP32_C6_LIBRARY_6_SOT65P210X110-3N
- R1, R17, R18, R1_EP_DR, R1_USB, R2, R2_EP_DR, R2_USB, R4, R5, R7, R8, R9, R_PWR_EPD, R_TYPE_SEL: device InkTime_v5:CPF0201D7K68C1_0201 -> InkTime_v5v3:CPF0201D7K68C1_0201
- SJ1: device InkTime_v5:ESP32_C6_LIBRARY_7_JUMPER_SJ -> InkTime_v5v3:ESP32_C6_LIBRARY_7_JUMPER_SJ
- SW_DN, SW_ENT, SW_UP: device InkTime_v5v2:2025-10-22_07-23-44_LIBRARY_SW_EVP-AKE31A_PAN -> InkTime_v5v3:2025-10-22_07-23-44_LIBRARY_SW_EVP-AKE31A_PAN
- TP_3.3V, TP_3V3, TP_BAT_GND, TP_GND, TP_RESET, TP_SCL, TP_SDA, TP_SWDCLK, TP_SWDIO, TP_SWO, TP_VBAT, TP_VREG: device InkTime_v5:HECTOR_WATCH_1_TP20R -> InkTime_v5v3:HECTOR_WATCH_1_TP20R
- U1: device InkTime_v5:NORDIC_NRF_4_AQFN50P700X700X85_HS-74N -> InkTime_v5v3:NORDIC_NRF_4_AQFN50P700X700X85_HS-74N
- U3: device InkTime_v5:ESP32_C6_LIBRARY_SON50P200X200X80-9N -> InkTime_v5v3:ESP32_C6_LIBRARY_SON50P200X200X80-9N
- X1: device InkTime_v5:NORDIC_NRF_BT-XTAL_2016_N -> InkTime_v5v3:NORDIC_NRF_BT-XTAL_2016_N
- X2: device InkTime_v5:NORDIC_NRF_1_XTAL_3215_N -> InkTime_v5v3:NORDIC_NRF_1_XTAL_3215_N
